File: PowerModule/power_module/power_module.kicad_pcb (KiCad board)
At the start: 2 copper layers, 41 x 41 mm, 1 part

Commit message: update
Parts:
- added C1: 0.1uF/275V, power_module:CAP_MKP64, F.Cu at (143.5, 66.0)
- added C2: CP, Capacitor_THT:CP_Radial_D6.3mm_P2.50mm, F.Cu at (116.8, 44.5)
- added F1: 0.5A/250V, power_module:FUZE3x10, F.Cu at (139.7, 54.6)
- added L1: 10mH, power_module:inductor, F.Cu at (133.3, 71.1)
- added RV1: 10D561, power_module:Varistor, F.Cu at (133.3, 58.4)
- moved PS1 5.39 mm to (118.1, 67.3), turned to 90 degrees
Other:
- board size 41 x 41 mm -> 41 x 41.9 mm
