File: ESP2866_Dimmer/LHD-45A.kicad_sch (KiCad schematic)
At the start: 4 parts, among them J10 Conn_01x04_Male, J8 Conn_01x04_Male, J9 Conn_01x04_Male, U9 LDH-45A-350

Commit message: Окремий проект для плати драйверу.
Parts:
- U9: footprint (none) -> dimmer:LDH-45A
Connections:
- net at U9. (Vout-): now also J10.2 (Pin_2)
Changed lines of the file:
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@@
     (property "Reference" "U9" (id 0) (at 144.145 49.53 0))
     (property "Value" "LDH-45A-350" (id 1) (at 144.145 52.07 0))
-    (property "Footprint" "" (id 2) (at 143.51 45.72 0)
+    (property "Footprint" "dimmer:LDH-45A" (id 2) (at 143.51 45.72 0)
       (effects (font (size 1.27 1.27)) hide)
     )
