File: ESP2866_Dimmer/top_plate_dimmer/top_plate_dimmer.kicad_pcb (KiCad board)
At the start: 2 copper layers, 60.1 x 98 mm, 17 parts, among them J1 Conn_01x06, J2 Conn_01x16, K1 SILxx-1Axx-71x, Q1 2N3904, Q2 2N3904, U1 LDH-45A-350

Commit message: Beta version (fixed)
Parts:
- removed the REF** at (122.1, 124.0)
- removed the REF** at (177.1, 31.1)
- removed the REF** at (177.1, 124.0)
- removed the REF** at (122.1, 31.1)
- added REF**: MountingHole_3mm, MountingHole:MountingHole_3mm, F.Cu at (177.1, 31.1)
- added REF**: MountingHole_3mm, MountingHole:MountingHole_3mm, F.Cu at (177.1, 124.1)
- added REF**: MountingHole_3mm, MountingHole:MountingHole_3mm, F.Cu at (122.1, 124.1)
- added REF**: MountingHole_3mm, MountingHole:MountingHole_3mm, F.Cu at (122.1, 31.1)
Other:
- board size 60.1 x 98 mm -> 60 x 98 mm
