File: ESP2866_Dimmer/dimmer/dimmer.kicad_pcb (KiCad board)
At the start: 2 copper layers, 84 x 100 mm, 33 parts, among them J1 Conn_01x03_Male, J2 Screw_Terminal_01x02, J3 Screw_Terminal_01x04, J4 Conn_01x08, J5 Conn_01x03_Male, J6 Conn_01x03_Male, J7 Screw_Terminal_01x02, J8 Conn_01x06, SW1 SW_Push, SW2 SW_Push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

Commit message: Next update
Parts:
- removed J5: Conn_01x03_Male, Connector_JST:JST_EH_B3B-EH-A_1x03_P2.50mm_Vertical
- added J9: Conn_01x16_Female, Connector_PinSocket_2.54mm:PinSocket_1x16_P2.54mm_Vertical, F.Cu at (36.1, 133.9)
- added Q1: 2N3904, Package_TO_SOT_THT:TO-92_Inline, F.Cu at (24.5, 102.8)
- added R10: 10k, Resistor_SMD:R_1206_3216Metric_Pad1.30x1.75mm_HandSolder, F.Cu at (58.3, 108.8)
- added R11: 165, Resistor_SMD:R_1206_3216Metric_Pad1.30x1.75mm_HandSolder, F.Cu at (41.6, 113.8)
- added R12: 470, Resistor_SMD:R_1206_3216Metric_Pad1.30x1.75mm_HandSolder, F.Cu at (58.5, 97.5)
- added R8: 10k, Resistor_SMD:R_1206_3216Metric_Pad1.30x1.75mm_HandSolder, F.Cu at (59.8, 114.1)
- added R9: 10k, Resistor_SMD:R_1206_3216Metric_Pad1.30x1.75mm_HandSolder, F.Cu at (59.0, 83.8)
- J1: value Conn_01x03_Male -> Screw_Terminal_01x04; footprint Connector_JST:JST_EH_B3B-EH-A_1x03_P2.50mm_Vertical -> dimmer:DG126-5.0-04P-14_Vertical
- J2: footprint Connector_JST:JST_NV_B02P-NV_1x02_P5.00mm_Vertical -> dimmer:DG126-5.0-02P-14_Vertical
- SW1: value SW_Push -> Reset
- SW2: value SW_Push -> Menu1
- SW3: value SW_Push -> Menu2
- SW4: value SW_Push -> Menu3
- SW5: value SW_Push -> Menu4
- U1: value L78L03_SOT89 -> AP1117-33; footprint Package_TO_SOT_SMD:SOT-89-3 -> Package_TO_SOT_SMD:SOT-223-3_TabPin2
- U3: value L78L05_SOT89 -> AP1117-50; footprint Package_TO_SOT_SMD:SOT-89-3 -> Package_TO_SOT_SMD:SOT-223-3_TabPin2
- moved J8 95.2 mm to (73.8, 150.8), turned to -90 degrees
- moved J4 94.0 mm to (69.0, 57.6), turned to -90 degrees
- moved J2 72.0 mm to (25.7, 139.3)
- moved J1 69.8 mm to (25.6, 78.9), turned to -90 degrees
- moved J7 69.6 mm to (25.6, 63.8)
- moved U1 47.6 mm to (48.2, 66.5)
- moved C2 35.7 mm to (54.3, 137.6)
- moved C3 23.3 mm to (47.8, 131.3)
- moved J3 20.2 mm to (25.6, 112.8)
- moved C1 16.3 mm to (41.0, 75.2)
- moved U3 8.66 mm to (62.5, 66.5)
Connections:
- J1 pad 3: GND -> /LIGHT_SENSOR
- U1 pad 1: +3V3 -> GND
- U1 pad 2: GND -> +3V3
- U3 pad 1: +5V -> GND
- U3 pad 2: GND -> +5V
- U6 pad 1: unconnected-(U6-Pad1) -> Net-(U6-Pad1)
- U6 pad 10: unconnected-(U6-Pad10) -> Net-(U6-Pad10)
- U6 pad 11: unconnected-(U6-Pad11) -> Net-(U6-Pad11)
- U6 pad 12: unconnected-(U6-Pad12) -> Net-(J9-Pad14)
- U6 pad 2: unconnected-(U6-Pad2) -> Net-(U6-Pad2)
- U6 pad 3: unconnected-(U6-Pad3) -> Net-(U6-Pad3)
- U6 pad 4: unconnected-(U6-Pad4) -> Net-(U6-Pad4)
- U6 pad 5: unconnected-(U6-Pad5) -> Net-(U6-Pad5)
- U6 pad 6: unconnected-(U6-Pad6) -> Net-(U6-Pad6)
- U6 pad 7: unconnected-(U6-Pad7) -> Net-(U6-Pad7)
- U6 pad 9: unconnected-(U6-Pad9) -> Net-(U6-Pad9)

Commit message: Beta version (fixed)
Parts:
- removed the REF** at (91.3, 150.6)
- removed the REF** at (91.3, 57.6)
- removed the REF** at (36.3, 150.6)
- removed the REF** at (36.3, 57.6)
- added R13: 10k, Resistor_SMD:R_1206_3216Metric_Pad1.30x1.75mm_HandSolder, F.Cu at (59.7, 93.5)
- added R14: 10k, Resistor_SMD:R_1206_3216Metric_Pad1.30x1.75mm_HandSolder, F.Cu at (63.7, 93.6)
- added REF**: MountingHole_3mm, MountingHole:MountingHole_3mm, F.Cu at (38.8, 140.5)
- added REF**: MountingHole_3mm, MountingHole:MountingHole_3mm, F.Cu at (91.4, 57.7)
- added REF**: MountingHole_3mm, MountingHole:MountingHole_3mm, F.Cu at (36.4, 57.7)
- added REF**: MountingHole_3mm, MountingHole:MountingHole_3mm, F.Cu at (89.2, 68.8)
- added REF**: MountingHole_3mm, MountingHole:MountingHole_3mm, F.Cu at (36.4, 150.7)
- added REF**: MountingHole_3mm, MountingHole:MountingHole_3mm, F.Cu at (89.2, 140.5)
- added REF**: MountingHole_3mm, MountingHole:MountingHole_3mm, F.Cu at (91.4, 150.7)
- added REF**: MountingHole_3mm, MountingHole:MountingHole_3mm, F.Cu at (38.8, 68.8)
- added RV1: R_Potentiometer, dimmer:TRIM_3296W-1-203, F.Cu at (28.3, 135.6)
- moved U1 57.4 mm to (79.8, 114.4), turned to -90 degrees
- moved R9 47.7 mm to (45.9, 129.8), turned to 90 degrees
- moved C2 40.8 mm to (81.0, 106.7)
- moved R5 39.9 mm to (61.2, 82.0)
- moved R3 38.0 mm to (61.3, 89.2)
- moved SW3 37.6 mm to (104.4, 140.1)
- moved SW5 37.3 mm to (104.4, 129.9)
- moved SW4 36.8 mm to (104.4, 119.7)
- moved SW2 36.4 mm to (104.4, 109.5)
- moved U3 33.0 mm to (48.1, 96.1), turned to 90 degrees
- moved R4 31.2 mm to (61.2, 85.9)
- moved R6 27.9 mm to (61.6, 101.4)
- moved R2 26.8 mm to (95.4, 77.7)
- moved R12 26.3 mm to (32.1, 97.2), turned to 90 degrees
- moved C3 25.9 mm to (48.0, 105.4), turned to 180 degrees
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Connections:
- J9 pad 15: 5V -> +5V
- J9 pad 2: 5V -> +5V
- R10 pad 1: 5V -> +5V
- R8 pad 1: 5V -> +5V
- R9 pad 1: 5V -> +5V
- U4 pad 8: 5V -> +5V
- U5 pad 1: unconnected-(U5-Pad1) -> Net-(R14-Pad2)
- U5 pad 10: unconnected-(U5-Pad10) -> /LED_ON_RELE
- U5 pad 16: 5V -> +5V
- U5 pad 2: unconnected-(U5-Pad2) -> Net-(R13-Pad2)
- U6 pad 16: 5V -> +5V
Routing:
- net +5V: track 0.00 -> 176.6 mm, vias 0 -> 3
- net +3V3: track 0.00 -> 119.9 mm, vias 0 -> 2
- net +12V: track 0.00 -> 118.6 mm, vias 0 -> 3
- net /DOWN: track 0.00 -> 92.5 mm, vias 0 -> 1
- net /SDA: track 0.00 -> 91.6 mm
- net /SCL: track 0.00 -> 86.4 mm, vias 0 -> 3
- net /UP: track 0.00 -> 79.1 mm, vias 0 -> 1
- net /LIGHT_SENSOR: track 0.00 -> 69.8 mm, vias 0 -> 2
- net /ON_OFF: track 0.00 -> 69.3 mm, vias 0 -> 3
- net /MENU2: track 0.00 -> 67.1 mm, vias 0 -> 2
- net /MOVE_SENSOR: track 0.00 -> 61.4 mm
- net /LED_ON_RELE: track 0.00 -> 60.1 mm, vias 0 -> 1
- net Net-(J2-Pad1): track 0.00 -> 57.8 mm
- net /MENU4: track 0.00 -> 55.1 mm, vias 0 -> 2
- net /PWM_OUT: track 0.00 -> 49.2 mm, vias 0 -> 1
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- added copper zone on B.Cu, net GND
- added copper zone on F.Cu, net GND
Other:
- board size 84 x 100 mm -> 84 x 100.2 mm

Commit message: Beta2
Parts:
- added C4: 100n, Capacitor_SMD:C_1206_3216Metric_Pad1.33x1.80mm_HandSolder, F.Cu at (49.4, 79.7)
- added C5: 100n 100v, Capacitor_SMD:C_1206_3216Metric_Pad1.33x1.80mm_HandSolder, F.Cu at (43.9, 60.9)
- added D1: BZV55-12V, Diode_SMD:D_MiniMELF, F.Cu at (49.5, 75.8)
- added FLASH: Flash, Button_Switch_THT:SW_PUSH_6mm, F.Cu at (71.3, 126.0)
- added Q2: DMG1012T, Package_TO_SOT_SMD:SOT-523, F.Cu at (69.8, 108.5)
- added Q3: DMG1012T, Package_TO_SOT_SMD:SOT-523, F.Cu at (74.0, 108.5)
- added Q4: FDD4141, dpak:DPAK-3, F.Cu at (49.6, 66.9)
- added R15: 10k, Resistor_SMD:R_1206_3216Metric_Pad1.30x1.75mm_HandSolder, F.Cu at (81.9, 124.3)
- added R16: 10k, Resistor_SMD:R_1206_3216Metric_Pad1.30x1.75mm_HandSolder, F.Cu at (85.4, 112.4)
- added R17: 10k, Resistor_SMD:R_1206_3216Metric_Pad1.30x1.75mm_HandSolder, F.Cu at (95.5, 113.1)
- added R18: 10k, Resistor_SMD:R_1206_3216Metric_Pad1.30x1.75mm_HandSolder, F.Cu at (95.5, 143.4)
- added R19: 10k, Resistor_SMD:R_1206_3216Metric_Pad1.30x1.75mm_HandSolder, F.Cu at (95.5, 123.1)
- added R20: 10k, Resistor_SMD:R_1206_3216Metric_Pad1.30x1.75mm_HandSolder, F.Cu at (95.5, 132.5)
- added R21: 10k, Resistor_SMD:R_1206_3216Metric_Pad1.30x1.75mm_HandSolder, F.Cu at (68.0, 115.7)
- added R22: 10k, Resistor_SMD:R_1206_3216Metric_Pad1.30x1.75mm_HandSolder, F.Cu at (72.4, 115.7)
- added R23: 12K 1%, Resistor_SMD:R_1206_3216Metric, F.Cu at (43.6, 75.7)
- REF** (x4): value MountingHole_3mm -> MountingHole_3.5mm; footprint MountingHole:MountingHole_3mm -> MountingHole:MountingHole_3.5mm
- moved R12 8.14 mm to (40.3, 96.6)
Connections:
- J7 pad 1: +12V -> /+12vInput
- SW2 pad 1: GND -> +3V3
- SW3 pad 1: GND -> +3V3
- SW4 pad 1: GND -> +3V3
- SW5 pad 1: GND -> +3V3
- U2 pad 17: unconnected-(U2-Pad17) -> Net-(U2-Pad17)
- U2 pad 18: unconnected-(U2-Pad18) -> Net-(U2-Pad18)
- U2 pad 19: /SDA -> /SDA3V
- U2 pad 20: /SCL -> /SCL3V
- U4 pad 1: unconnected-(U4-Pad1) -> GND
- U4 pad 2: unconnected-(U4-Pad2) -> GND
- U4 pad 3: unconnected-(U4-Pad3) -> GND
Routing:
- net +3V3: track 119.9 -> 258.3 mm, vias 2 -> 3
- net Net-(U2-Pad18): track 0.00 -> 46.7 mm, vias 0 -> 2
- net /SDA3V: track 0.00 -> 31.8 mm
- net /SCL3V: track 0.00 -> 29.9 mm
- net +12V: track 118.6 -> 92.2 mm
- net /+12vInput: track 0.00 -> 25.5 mm
- net /SDA: track 91.6 -> 73.8 mm
- net Net-(U2-Pad17): track 0.00 -> 17.3 mm, vias 0 -> 2
- net /SCL: track 86.4 -> 70.9 mm, vias 3 -> 5
- net Net-(C4-Pad2): track 0.00 -> 11.7 mm
- net /MENU4: track 55.1 -> 60.0 mm
- net /MENU2: track 67.1 -> 71.8 mm
- net +5V: track 176.6 -> 172.9 mm
- net /MENU1: track 48.6 -> 50.8 mm
- net /MENU3: track 38.4 -> 40.4 mm
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Other:
- board text added: "+12V"
- board text added: "- + LED"
- board text added: "GND"
- board text added: "GND DOWN UP +3.3"
- board text added: "GND LIGHT MOVE +3.3"

Commit message: Fix eeror in connection
Parts:
- renumbered FLASH to SW6
Connections:
- Q2 pad 1: GND -> +3V3
- Q3 pad 1: GND -> +3V3
- R13 pad 1: 5V -> +5V
- R14 pad 1: 5V -> +5V
Routing:
- net +3V3: track 258.3 -> 279.1 mm
- net +5V: track 172.9 -> 182.1 mm
- net 5V: track 4.09 -> 0.00 mm
- net GND: track 1.45 -> 0.00 mm, vias 47 -> 46
