File: ESP2866_Dimmer/dimmer/dimmer.kicad_sch (KiCad schematic)
At the start: 43 parts, among them J1 Conn_01x03_Male, J2 Screw_Terminal_01x02, J3 Conn_01x03_Male, J4 Conn_01x04_Male, J5 Screw_Terminal_01x04, J6 Screw_Terminal_01x02, K1 TIANBO-HJR-4102-L, Q1 2N3904, SW1 SW_Push, U1 LDH-45A-350, U2 B1203S-1WR3, U3 ESP-12E, U4 LTV-354T, U5 LTV-354T, U6 LTV-354T, U7 LTV-354T, U8 LTV-354T, U9 L78L05_SOT89

Commit message: Update next.
Parts:
- removed J5: Screw_Terminal_01x04, Connector_JST:JST_NV_B04P-NV_1x04_P5.00mm_Vertical, symbol Connector:Screw_Terminal_01x04
- added J5, J6: Screw_Terminal_01x02, Connector_JST:JST_NV_B02P-NV_1x02_P5.00mm_Vertical, symbol Connector:Screw_Terminal_01x02
- J2: footprint TerminalBlock_MetzConnect:TerminalBlock_MetzConnect_Type011_RT05502HBWC_1x02_P5.00mm_Horizontal -> Connector_JST:JST_NV_B02P-NV_1x02_P5.00mm_Vertical
- renumbered J6 to J7
Connections:
- net GND2: now also J6.2 (Pin_2)
- net at R11.2: now also J5.1 (Pin_1)
- net at R15.2: now also J5.2 (Pin_2)
- net at R20.2: now also J6.1 (Pin_1)
Changed lines of the file:
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@@
   (symbol (lib_id "Connector:Screw_Terminal_01x02") (at 33.02 160.02 0) (mirror y) (unit 1)
     (in_bom yes) (on_board yes)
-    (property "Reference" "J6" (id 0) (at 35.1028 154.5082 0))
+    (property "Reference" "J7" (id 0) (at 35.1028 154.5082 0))
     (property "Value" "Screw_Terminal_01x02" (id 1) (at 35.1028 156.8196 0))
     (property "Footprint" "Connector_JST:JST_NV_B02P-NV_1x02_P5.00mm_Vertical" (id 2) (at 33.02 160.02 0)
@@
     (pin "1")
   )
+  (symbol (lib_id "Connector:Screw_Terminal_01x02") (at 170.18 100.33 0) (mirror y) (unit 1)
+    (in_bom yes) (on_board yes)
+    (property "Reference" "J6" (id 0) (at 172.2628 94.8182 0))
+    (property "Value" "Screw_Terminal_01x02" (id 1) (at 172.2628 97.1296 0))
+    (property "Footprint" "Connector_JST:JST_NV_B02P-NV_1x02_P5.00mm_Vertical" (id 2) (at 170.18 100.33 0)
+      (effects (font (size 1.27 1.27)) hide)
+    )
+    (property "Datasheet" "~" (id 3) (at 170.18 100.33 0)
+      (effects (font (size 1.27 1.27)) hide)
+    )
+    (pin "1")
+    (pin "2")
+  )
   (symbol (lib_id "power:+5V") (at 212.09 90.17 0) (unit 1)
     (in_bom yes) (on_board yes)
@@
     )
     (pin "1")
+  )
+  (symbol (lib_id "Connector:Screw_Terminal_01x02") (at 274.32 27.94 0) (unit 1)
+    (in_bom yes) (on_board yes)
+    (property "Reference" "J2" (id 0) (at 272.2372 22.4282 0))
+    (property "Value" "Screw_Terminal_01x02" (id 1) (at 272.2372 24.7396 0))
+    (property "Footprint" "Connector_JST:JST_NV_B02P-NV_1x02_P5.00mm_Vertical" (id 2) (at 274.32 27.94 0)
+      (effects (font (size 1.27 1.27)) hide)
+    )
+    (property "Datasheet" "~" (id 3) (at 274.32 27.94 0)
+      (effects (font (size 1.27 1.27)) hide)
+    )
+    (pin "1")
+    (pin "2")
   )
   (symbol (lib_id "power:GNDPWR") (at 127 119.38 0) (unit 1)
@@
     (property "Datasheet" "http://optoelectronics.liteon.com/upload/download/DS70-2001-004/S_110_LTV-354T%2020140520.pdf" (id 3) (at 95.885 116.84 0)
       (effects (font (size 1.27 1.27)) (justify left) hide)
-    )
-    (pin "1")
-    (pin "2")
-    (pin "3")
-    (pin "4")
-  )
-  (symbol (lib_id "Connector:Screw_Terminal_01x04") (at 170.18 97.79 0) (mirror y) (unit 1)
-    (in_bom yes) (on_board yes) (fields_autoplaced)
-    (property "Reference" "J5" (id 0) (at 170.18 88.9 0))
-    (property "Value" "Screw_Terminal_01x04" (id 1) (at 170.18 91.44 0))
-    (property "Footprint" "Connector_JST:JST_NV_B04P-NV_1x04_P5.00mm_Vertical" (id 2) (at 170.18 97.79 0)
-      (effects (font (size 1.27 1.27)) hide)
-    )
-    (property "Datasheet" "~" (id 3) (at 170.18 97.79 0)
-      (effects (font (size 1.27 1.27)) hide)
     )
     (pin "1")
@@
     (pin "1")
   )
+  (symbol (lib_id "Connector:Screw_Terminal_01x02") (at 170.18 95.25 0) (mirror y) (unit 1)
+    (in_bom yes) (on_board yes)
+    (property "Reference" "J5" (id 0) (at 172.2628 89.7382 0))
+    (property "Value" "Screw_Terminal_01x02" (id 1) (at 172.2628 92.0496 0))
+    (property "Footprint" "Connector_JST:JST_NV_B02P-NV_1x02_P5.00mm_Vertical" (id 2) (at 170.18 95.25 0)
+      (effects (font (size 1.27 1.27)) hide)
+    )
+    (property "Datasheet" "~" (id 3) (at 170.18 95.25 0)
+      (effects (font (size 1.27 1.27)) hide)
+    )
+    (pin "1")
+    (pin "2")
+  )
   (symbol (lib_id "power:GND") (at 86.36 31.75 0) (unit 1)
     (in_bom yes) (on_board yes)
@@
     (pin "2")
   )
-  (symbol (lib_id "Connector:Screw_Terminal_01x02") (at 274.32 27.94 0) (unit 1)
-    (in_bom yes) (on_board yes) (fields_autoplaced)
-    (property "Reference" "J2" (id 0) (at 276.86 27.9399 0)
-      (effects (font (size 1.27 1.27)) (justify left))
-    )
-    (property "Value" "Screw_Terminal_01x02" (id 1) (at 276.86 30.4799 0)
-      (effects (font (size 1.27 1.27)) (justify left))
-    )
-    (property "Footprint" "TerminalBlock_MetzConnect:TerminalBlock_MetzConnect_Type011_RT05502HBWC_1x02_P5.00mm_Horizontal" (id 2) (at 274.32 27.94 0)
-      (effects (font (size 1.27 1.27)) hide)
-    )
-    (property "Datasheet" "~" (id 3) (at 274.32 27.94 0)
-      (effects (font (size 1.27 1.27)) hide)
-    )
-    (pin "1")
-    (pin "2")
-  )
   (symbol (lib_id "power:GNDPWR") (at 49.53 162.56 0) (unit 1)
     (in_bom yes) (on_board yes) (fields_autoplaced)
@@
       (reference "J1") (unit 1) (value "Conn_01x03_Male") (footprint "Connector_JST:JST_EH_B3B-EH-A_1x03_P2.50mm_Vertical")
     )
-    (path "/f1ce9232-74d9-405b-8822-05d2b14c73e1"
-      (reference "J2") (unit 1) (value "Screw_Terminal_01x02") (footprint "TerminalBlock_MetzConnect:TerminalBlock_MetzConnect_Type011_RT05502HBWC_1x02_P5.00mm_Horizontal")
+    (path "/377a03da-7f35-42f3-ab79-a2dc1b74733f"
+      (reference "J2") (unit 1) (value "Screw_Terminal_01x02") (footprint "Connector_JST:JST_NV_B02P-NV_1x02_P5.00mm_Vertical")
     )
     (path "/8ca2c50b-bf3a-438b-a227-f2ee9e498fd9"
@@
       (reference "J4") (unit 1) (value "Conn_01x04_Male") (footprint "Connector_Stocko:Stocko_MKS_1654-6-0-404_1x4_P2.50mm_Vertical")
     )
-    (path "/4d95ec5d-045d-4cf9-a97c-3034968cae45"
-      (reference "J5") (unit 1) (value "Screw_Terminal_01x04") (footprint "Connector_JST:JST_NV_B04P-NV_1x04_P5.00mm_Vertical")
+    (path "/953d45d5-e11a-4df6-a8ea-bd278753d364"
+      (reference "J5") (unit 1) (value "Screw_Terminal_01x02") (footprint "Connector_JST:JST_NV_B02P-NV_1x02_P5.00mm_Vertical")
+    )
+    (path "/2e924d2d-94f7-4a0f-8528-9d6e8f6bb0eb"
+      (reference "J6") (unit 1) (value "Screw_Terminal_01x02") (footprint "Connector_JST:JST_NV_B02P-NV_1x02_P5.00mm_Vertical")
     )
     (path "/00000000-0000-0000-0000-00005eafc839"
-      (reference "J6") (unit 1) (value "Screw_Terminal_01x02") (footprint "Connector_JST:JST_NV_B02P-NV_1x02_P5.00mm_Vertical")
+      (reference "J7") (unit 1) (value "Screw_Terminal_01x02") (footprint "Connector_JST:JST_NV_B02P-NV_1x02_P5.00mm_Vertical")
     )
     (path "/dcc8b3c7-e00a-4c96-92c3-7cf68574fa70"

Commit message: Big Update.
Parts:
- removed D1: 1N4003, Diode_SMD:D_SMA, symbol Diode:1N4003
- removed F1: Fuse, Fuse:Fuse_2920_7451Metric_Pad2.10x5.45mm_HandSolder, symbol Device:Fuse
- removed J4: Conn_01x04_Male, Connector_Stocko:Stocko_MKS_1654-6-0-404_1x4_P2.50mm_Vertical, symbol Connector:Conn_01x04_Male
- removed J5, J6: Screw_Terminal_01x02, Connector_JST:JST_NV_B02P-NV_1x02_P5.00mm_Vertical, symbol Connector:Screw_Terminal_01x02
- removed K1: TIANBO-HJR-4102-L, Relay_THT:Relay_SPDT_HJR-4102, symbol Relay:TIANBO-HJR-4102-L
- removed Q1: 2N3904, Package_TO_SOT_THT:TO-92_Inline, symbol Transistor_BJT:2N3904
- removed R10, R12, R16: 330, Resistor_SMD:R_1206_3216Metric_Pad1.30x1.75mm_HandSolder, symbol Device:R
- removed R11, R15, R20, R3, R5: 0, Resistor_SMD:R_1206_3216Metric_Pad1.30x1.75mm_HandSolder, symbol Device:R
- removed R13: 240, Resistor_SMD:R_1206_3216Metric_Pad1.30x1.75mm_HandSolder, symbol Device:R
- removed R17: 1k, Resistor_SMD:R_1206_3216Metric_Pad1.30x1.75mm_HandSolder, symbol Device:R
- removed R19, R8: 165, Resistor_SMD:R_1206_3216Metric_Pad1.30x1.75mm_HandSolder, symbol Device:R
- removed R4: 110, Resistor_SMD:R_1206_3216Metric_Pad1.30x1.75mm_HandSolder, symbol Device:R
- removed U1: LDH-45A-350, dimmer:LDH-45A, symbol dimmer_lib:LDH-45A-350
- removed U2: B1203S-1WR3, dimmer:B1203-1WR3, symbol dimmer_lib:B1205S-1WR3
- removed U4, U5, U6, U7, U8: LTV-354T, Package_SO:SO-4_4.4x3.6mm_P2.54mm, symbol Isolator:LTV-354T
- added J10: Conn_01x16_Male, symbol Connector:Conn_01x16_Male
- added J3: Screw_Terminal_01x04, Connector_JST:JST_NV_B04P-NV_1x04_P5.00mm_Vertical, symbol Connector:Screw_Terminal_01x04
- added J4: Conn_01x08, Connector_PinSocket_1.27mm:PinSocket_1x16_P1.27mm_Vertical, symbol Connector_Generic:Conn_01x16
- added J6: Conn_01x03_Male, Connector_JST:JST_EH_B3B-EH-A_1x03_P2.50mm_Vertical, symbol Connector:Conn_01x03_Male
- added J8: Conn_01x06, Connector_PinSocket_1.27mm:PinSocket_1x14_P1.27mm_Vertical, symbol Connector_Generic:Conn_01x14
- added J9: Conn_01x16_Female, symbol Connector:Conn_01x16_Female
- added SW2, SW3, SW4, SW5: SW_Push, Button_Switch_THT:SW_PUSH_6mm, symbol Switch:SW_Push
- added U1: L78L03_SOT89, Package_TO_SOT_SMD:SOT-89-3, symbol Regulator_Linear:L78L05_SOT89
- added U4: 24LC01, Package_SO:SOIC-8_3.9x4.9mm_P1.27mm, symbol Memory_EEPROM:24LC01
- added U5, U6: PCF8574, Package_SO:SOIC-16W_7.5x10.3mm_P1.27mm, symbol Interface_Expansion:PCF8574
- added U7: LCD-20X4, symbol tinkerforge:LCD-20X4
- R3: renamed from R18; value 250 -> 10k
- R4: renamed from R14; value 250 -> 10k
- R5: renamed from R9; value 250 -> 10k
- R6: value 0 -> 10k
- R7: value 470 -> 10k
- renumbered J3 to J5, U3 to U2, U9 to U3
Connections:
- net GNDPWR is gone; now on net GND: C1.2, C3.2, J7.2 (Pin_2), U3.2 (GND)
- net +12V: now also J4.1 (Pin_1), J4.2 (Pin_2), J4.3 (Pin_3), J4.4 (Pin_4), J4.5 (Pin_5), J4.6 (Pin_6), U1.3 (IN)
- net +3V3: now also C2.1, U1.1 (OUT)
- net +5V: now also R6.1, J4.13 (Pin_13); no longer R6.2
- net DOWN: now also R5.2, J3.3 (Pin_3), U5.6 (P2); no longer U2.5 (GPIO14)
- net ESP_RX: now also J6.2 (Pin_2)
- net ESP_TX: now also J6.1 (Pin_1)
- net GND: now also J3.4 (Pin_4), J4.10 (Pin_10), J4.11 (Pin_11), J4.12 (Pin_12), J4.7 (Pin_7), J4.8 (Pin_8), J4.9 (Pin_9), J6.3 (Pin_3), SW2.1, SW3.1, SW4.1, SW5.1, U1.2 (GND), U4.4 (GND), U5.3 (A2), U5.8 (VSS), U6.8 (VSS)
- net LED_ON_RELE: now also J4.14 (Pin_14)
- net LIGHT_SENSOR: now also U5.7 (P3); no longer U2.6 (GPIO12)
- net MOVE_SENSOR: now also U5.9 (P4); no longer U2.20 (GPIO5)
- net ON_OFF: now also R3.2, J3.1 (Pin_1), U5.4 (P0); no longer U2.12 (GPIO10)
- net UP: now also R4.2, J3.2 (Pin_2), U5.5 (P1); no longer U2.7 (GPIO13)
- net MENU3: now reaches U2.16 (GPIO15)
- net MENU3: now also SW4.2
- net MENU4: now reaches U2.4 (GPIO16)
- net MENU4: now also SW5.2
- net at J2.1 (Pin_1): now also J8.1 (Pin_1), J8.2 (Pin_2), J8.3 (Pin_3), J8.4 (Pin_4), J8.5 (Pin_5), J8.6 (Pin_6), J8.7 (Pin_7)
- net at J2.2 (Pin_2): now also J8.10 (Pin_10), J8.11 (Pin_11), J8.12 (Pin_12), J8.13 (Pin_13), J8.14 (Pin_14), J8.8 (Pin_8), J8.9 (Pin_9)
- net SCL: now reaches R7.2
- net SCL: now also U2.20 (GPIO5), U4.6 (SCL), U5.14 (SCL), U6.14 (SCL)
- net PWM renamed SDA
- net SDA: now also R6.2, U4.5 (SDA), U5.15 (SDA), U6.15 (SDA)
- new net: J10.1 (Pin_1), U7.1 (VSS)
- new net: J10.10 (Pin_10), U7.10 (DB3)
- new net: J10.11 (Pin_11), U7.11 (DB4)
- new net: J10.12 (Pin_12), U7.12 (DB5)
- new net: J10.13 (Pin_13), U7.13 (DB6)
- new net: J10.14 (Pin_14), U7.14 (DB7)
- new net: J10.15 (Pin_15), U7.15 (A)
- new net: J10.16 (Pin_16), U7.16 (K)
- new net: J10.2 (Pin_2), U7.2 (VDD)
- new net: J10.3 (Pin_3), U7.3 (V0)
- new net: J10.4 (Pin_4), U7.4 (RS)
- new net: J10.5 (Pin_5), U7.5 (R/W)
- new net: J10.6 (Pin_6), U7.6 (E)
- new net: J10.7 (Pin_7), U7.7 (DB0)
- new net: J10.8 (Pin_8), U7.8 (DB1)
- new net: J10.9 (Pin_9), U7.9 (DB2)
- new net 5V: U4.8 (VCC), U5.16 (VDD), U6.16 (VDD)
- new net MENU1: SW2.2, U2.7 (GPIO13)
- new net MENU2: SW3.2, U2.5 (GPIO14)
- new net PWM_OUT: J4.16 (Pin_16), U2.6 (GPIO12)
Other:
- moved on the sheet: C3, J2, J7, R3, R4, R5, U3

Commit message: Next update
Parts:
- removed J1, J5: Conn_01x03_Male, Connector_JST:JST_EH_B3B-EH-A_1x03_P2.50mm_Vertical, symbol Connector:Conn_01x03_Male
- removed U1: L78L03_SOT89, Package_TO_SOT_SMD:SOT-89-3, symbol Regulator_Linear:L78L05_SOT89
- removed U3: L78L05_SOT89, Package_TO_SOT_SMD:SOT-89-3, symbol Regulator_Linear:L78L05_SOT89
- added J1: Screw_Terminal_01x04, Connector_JST:JST_NV_B04P-NV_1x04_P5.00mm_Vertical, symbol Connector:Screw_Terminal_01x04
- added Q1: 2N3904, Package_TO_SOT_THT:TO-92_Inline, symbol Transistor_BJT:2N3904
- added R10, R8, R9: 10k, Resistor_SMD:R_1206_3216Metric_Pad1.30x1.75mm_HandSolder, symbol Device:R
- added R11: 165, Resistor_SMD:R_1206_3216Metric_Pad1.30x1.75mm_HandSolder, symbol Device:R
- added R12: 470, Resistor_SMD:R_1206_3216Metric_Pad1.30x1.75mm_HandSolder, symbol Device:R
- added RV1: R_Potentiometer, symbol Device:R_Potentiometer
- added U1: AP1117-33, Package_TO_SOT_SMD:SOT-223-3_TabPin2, symbol Regulator_Linear:AP1117-33
- added U3: AP1117-50, Package_TO_SOT_SMD:SOT-223-3_TabPin2, symbol Regulator_Linear:AP1117-50
- J10, U7: now left out of the parts list
- J9: footprint (none) -> Connector_PinSocket_2.54mm:PinSocket_1x16_P2.54mm_Vertical
- SW1: value SW_Push -> Reset
- SW2: value SW_Push -> Menu1
- SW3: value SW_Push -> Menu2
- SW4: value SW_Push -> Menu3
- SW5: value SW_Push -> Menu4
Connections:
- net +12V: now also U1.3 (VI), U3.3 (VI)
- net +3V3: now also J1.1 (Pin_1), U1.2 (VO)
- net +5V: now also R12.1, U3.2 (VO)
- net 5V: now also J9.15 (Pin_15), J9.2 (Pin_2), R10.1, R8.1, R9.1, RV1.1
- net GND: now also J9.1 (Pin_1), J1.4 (Pin_4), Q1.1 (E), RV1.3, U1.1 (GND), U3.1 (GND)
- net LIGHT_SENSOR: now also J1.3 (Pin_3)
- net MOVE_SENSOR: now also J1.2 (Pin_2)
- net at J9.11 (Pin_11): now also U6.9 (P4)
- net at J9.12 (Pin_12): now also U6.10 (P5)
- net at J9.13 (Pin_13): now also U6.11 (P6)
- net at J9.14 (Pin_14): now also U6.12 (P7)
- net KATHODE: now reaches J9.16 (Pin_16)
- net KATHODE: now also Q1.3 (C), R12.2
- net at J9.3 (Pin_3): now also RV1.2
- net at J9.4 (Pin_4): now also U6.4 (P0)
- net at J9.5 (Pin_5): now also U6.5 (P1)
- net at J9.6 (Pin_6): now also U6.6 (P2)
- net at U6.1 (A0): now also R10.2
- net at U6.2 (A1): now also R9.2
- net at U6.3 (A2): now also R8.2
- net at U6.7 (P3): now also R11.1
- new net: Q1.2 (B), R11.2
Other:
- moved on the sheet: J10, J3, J9, R3, R4, R5, R6, R7, U5, U6, U7

Commit message: Beta version (fixed)
Parts:
- added R13, R14: 10k, Resistor_SMD:R_1206_3216Metric_Pad1.30x1.75mm_HandSolder, symbol Device:R
- J1: footprint Connector_JST:JST_NV_B04P-NV_1x04_P5.00mm_Vertical -> dimmer:DG126-5.0-04P-14_Vertical
- J2: footprint Connector_JST:JST_NV_B02P-NV_1x02_P5.00mm_Vertical -> dimmer:DG126-5.0-02P-14_Vertical
Connections:
- net +5V: now also J9.15 (Pin_15), J9.2 (Pin_2), R10.1, R8.1, R9.1, RV1.1, U4.8 (VCC), U5.16 (VDD), U6.16 (VDD)
- net 5V: now also R13.1, R14.1; no longer J9.15 (Pin_15), J9.2 (Pin_2), R10.1, R8.1, R9.1, RV1.1, U4.8 (VCC), U5.16 (VDD), U6.16 (VDD)
- net LED_ON_RELE: now also U5.10 (P5)
- net at U5.1 (A0): now also R14.2
- net at U5.2 (A1): now also R13.2

Commit message: Beta2
Parts:
- added C4: 100n, Capacitor_SMD:C_1206_3216Metric_Pad1.33x1.80mm_HandSolder, symbol Device:C
- added C5: 100n 100v, Capacitor_SMD:C_1206_3216Metric_Pad1.33x1.80mm_HandSolder, symbol Device:C
- added D1: BZV55-12V, Diode_SMD:D_MiniMELF, symbol Diode:BZX84Cxx
- added Q2, Q3: DMG1012T, Package_TO_SOT_SMD:SOT-523, symbol Transistor_FET:DMG1012T
- added Q4: FDD4141, dpak:DPAK-3, symbol Transistor_FET:DMP3013SFV
- added R15, R16, R17, R18, R19, R20, R21, R22: 10k, Resistor_SMD:R_1206_3216Metric_Pad1.30x1.75mm_HandSolder, symbol Device:R
- added R23: 12K 1%, Resistor_SMD:R_1206_3216Metric, symbol Device:R
- added SW6: Flash, Button_Switch_THT:SW_PUSH_6mm, symbol Switch:SW_Push
Connections:
- net +12V: now also C4.1, D1.1 (K), Q4.3 (S); no longer J7.1 (Pin_1)
- net +3V3: now also SW2.1, SW3.1, SW4.1, SW5.1, R15.1, R16.1, R21.1, R22.1
- net GND: now also U4.1 (A0), U4.2 (A1), U4.3 (A2), C5.2, Q2.1 (G), Q3.1 (G), R17.2, R18.2, R19.2, R20.2, R23.2, SW6.2; no longer SW2.1, SW3.1, SW4.1, SW5.1
- net MENU1: now also R17.1
- net MENU2: now also R18.1
- net MENU3: now also R19.1
- net MENU4: now also R20.1
- net SCL: now also Q3.3 (D); no longer U2.20 (GPIO5)
- net SDA: now also Q2.3 (D); no longer U2.19 (GPIO4)
- net at U2.17 (GPIO2): now also R16.2
- net at U2.18 (GPIO0): now also R15.2, SW6.1
- new net: C4.2, D1.2 (A), Q4.1 (G), R23.1
- new net +12vInput: C5.1, J7.1 (Pin_1), Q4.2 (D)
- new net SCL3V: Q3.2 (S), R22.2, U2.20 (GPIO5)
- new net SDA3V: Q2.2 (S), R21.2, U2.19 (GPIO4)
Other:
- moved on the sheet: J1

Commit message: Fix eeror in connection
Connections:
- net 5V is gone; now on net +5V: R13.1, R14.1
- net +3V3: now also Q2.1 (G), Q3.1 (G)
- net GND: no longer Q2.1 (G), Q3.1 (G)
Changed lines of the file:
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@@
   (junction (at 226.06 21.59) (diameter 0) (color 0 0 0 0)
   )
+  (junction (at 144.78 71.12) (diameter 0) (color 0 0 0 0)
+  )
   (junction (at 190.5 138.43) (diameter 1.016) (color 0 0 0 0)
   )
@@
   (junction (at 279.4 25.4) (diameter 0) (color 0 0 0 0)
   )
+  (junction (at 78.74 85.09) (diameter 0) (color 0 0 0 0)
+  )
   (junction (at 46.99 34.29) (diameter 0) (color 0 0 0 0)
   )
@@
   )
   (junction (at 208.28 73.66) (diameter 0) (color 0 0 0 0)
+  )
+  (junction (at 121.92 85.09) (diameter 0) (color 0 0 0 0)
   )
   (junction (at 279.4 27.94) (diameter 0) (color 0 0 0 0)
@@
     (stroke (width 0) (type default) (color 0 0 0 0))
   )
+  (wire (pts (xy 95.25 87.63) (xy 95.25 85.09))
+    (stroke (width 0) (type default) (color 0 0 0 0))
+  )
   (wire (pts (xy 82.55 158.75) (xy 82.55 157.48))
     (stroke (width 0) (type default) (color 0 0 0 0))
@@
     (stroke (width 0) (type default) (color 0 0 0 0))
   )
+  (wire (pts (xy 138.43 85.09) (xy 121.92 85.09))
+    (stroke (width 0) (type default) (color 0 0 0 0))
+  )
   (wire (pts (xy 54.61 130.81) (xy 48.26 130.81))
     (stroke (width 0) (type default) (color 0 0 0 0))
@@
   )
   (wire (pts (xy 68.58 172.72) (xy 81.28 172.72))
+    (stroke (width 0) (type default) (color 0 0 0 0))
+  )
+  (wire (pts (xy 138.43 87.63) (xy 138.43 85.09))
     (stroke (width 0) (type default) (color 0 0 0 0))
   )
@@
   )
   (wire (pts (xy 39.37 157.48) (xy 43.18 157.48))
+    (stroke (width 0) (type default) (color 0 0 0 0))
+  )
+  (wire (pts (xy 95.25 85.09) (xy 78.74 85.09))
     (stroke (width 0) (type default) (color 0 0 0 0))
   )
@@
     (pin "1")
   )
+  (symbol (lib_id "power:+5V") (at 144.78 71.12 0) (unit 1)
+    (in_bom yes) (on_board yes)
+    (property "Reference" "#PWR0125" (id 0) (at 144.78 74.93 0)
+      (effects (font (size 1.27 1.27)) hide)
+    )
+    (property "Value" "+5V" (id 1) (at 145.161 66.7258 0))
+    (property "Footprint" "" (id 2) (at 144.78 71.12 0)
+      (effects (font (size 1.27 1.27)) hide)
+    )
+    (property "Datasheet" "" (id 3) (at 144.78 71.12 0)
+      (effects (font (size 1.27 1.27)) hide)
+    )
+    (pin "1")
+  )
   (symbol (lib_id "power:GND") (at 156.21 62.23 0) (unit 1)
     (in_bom yes) (on_board yes)
@@
     (pin "3")
   )
-  (symbol (lib_id "power:GND") (at 95.25 87.63 180) (unit 1)
-    (in_bom yes) (on_board yes)
-    (property "Reference" "#PWR0120" (id 0) (at 95.25 81.28 0)
-      (effects (font (size 1.27 1.27)) hide)
-    )
-    (property "Value" "GND" (id 1) (at 95.123 83.2358 0))
-    (property "Footprint" "" (id 2) (at 95.25 87.63 0)
-      (effects (font (size 1.27 1.27)) hide)
-    )
-    (property "Datasheet" "" (id 3) (at 95.25 87.63 0)
-      (effects (font (size 1.27 1.27)) hide)
-    )
-    (pin "1")
-  )
   (symbol (lib_id "Device:R") (at 163.83 25.4 0) (unit 1)
     (in_bom yes) (on_board yes)
@@
     (pin "1")
   )
-  (symbol (lib_id "power:GND") (at 138.43 87.63 180) (unit 1)
-    (in_bom yes) (on_board yes)
-    (property "Reference" "#PWR0115" (id 0) (at 138.43 81.28 0)
-      (effects (font (size 1.27 1.27)) hide)
-    )
-    (property "Value" "GND" (id 1) (at 138.303 83.2358 0))
-    (property "Footprint" "" (id 2) (at 138.43 87.63 0)
-      (effects (font (size 1.27 1.27)) hide)
-    )
-    (property "Datasheet" "" (id 3) (at 138.43 87.63 0)
-      (effects (font (size 1.27 1.27)) hide)
-    )
-    (pin "1")
-  )
   (symbol (lib_id "power:+5V") (at 38.1 123.19 0) (unit 1)
     (in_bom yes) (on_board yes)
@@
       (reference "#PWR0114") (unit 1) (value "GND") (footprint "")
     )
-    (path "/f084a9e7-a179-4d39-ba8a-389769eab4d5"
-      (reference "#PWR0115") (unit 1) (value "GND") (footprint "")
-    )
     (path "/aaf3b96a-c0fb-4c3f-828f-106254cfcefa"
       (reference "#PWR0116") (unit 1) (value "+3.3V") (footprint "")
@@
       (reference "#PWR0119") (unit 1) (value "+3.3V") (footprint "")
     )
-    (path "/7992dd3c-10af-46c7-bdfa-44ba09f110af"
-      (reference "#PWR0120") (unit 1) (value "GND") (footprint "")
-    )
     (path "/d77d241b-6f9f-420f-a177-394ba788b6c5"
       (reference "#PWR0121") (unit 1) (value "+3.3V") (footprint "")
@@
       (reference "#PWR0124") (unit 1) (value "GND") (footprint "")
     )
+    (path "/434a5981-015f-4644-af4b-a353a715d67a"
+      (reference "#PWR0125") (unit 1) (value "+5V") (footprint "")
+    )
     (path "/d313eb8e-cf40-4ef1-b0c2-bdf1a530763f"
